Commit message: feat: checkpoint unified navigation and plan four-package refactor
Add multi-floor navigation, shared foot motion, HMI algorithm selection,
adaptive step timing and footstep visualization updates.

Record the pre-refactor implementation and clarify the target package,
configuration, topic and URDF ownership in the new PRD. The dynamic-passage
timeout for F2-ROOM to F2-EAST remains unresolved; package migration is not
implemented. Historical execution evidence and build outputs were removed
at the user's request.

Validation: whitespace and Python/XML/YAML syntax checks. Simulation was
not rerun for this checkpoint.

File: sim_ws/src/sim_bringup/urdf/robot.urdf.xacro (robot description, xacro)
@@ -140,4 +140,13 @@
       <limit effort="${joint_effort}" velocity="${joint_speed}"/>
     </joint>
+    <link name="${side}_hip_yaw">
+      <inertial><mass value="0.001"/><inertia ixx="0.000001" ixy="0" ixz="0" iyy="0.000001" iyz="0" izz="0.000001"/></inertial>
+    </link>
+    <joint name="${side}_hip_yaw_joint" type="revolute">
+      <parent link="base_link"/><child link="${side}_hip_yaw"/>
+      <origin xyz="${shoulder_x} ${sign*shoulder_y} ${shoulder_z}"/>
+      <axis xyz="0 0 1"/>
+      <limit lower="-1.57" upper="1.57" effort="${joint_effort}" velocity="${leg_joint_speed}"/>
+    </joint>
     <link name="${side}_upper_leg">
       <xacro:box_parts sx="${leg_width}" sy="${leg_width}" sz="${upper_length}"
@@ -146,6 +155,6 @@
     <xacro:gazebo_color link="${side}_upper_leg" rgba="${limb_rgba}"/>
     <joint name="${side}_shoulder_joint" type="revolute">
-      <parent link="base_link"/><child link="${side}_upper_leg"/>
-      <origin xyz="${shoulder_x} ${sign*shoulder_y} ${shoulder_z}" rpy="0 ${shoulder_mount_pitch} 0"/>
+      <parent link="${side}_hip_yaw"/><child link="${side}_upper_leg"/>
+      <origin rpy="0 ${shoulder_mount_pitch} 0"/>
       <axis xyz="0 1 0"/>
       <limit lower="${-pitch_limit}" upper="${pitch_limit}" effort="${joint_effort}" velocity="${leg_joint_speed}"/>
